Commit message: add vision_detector

File: turtlebot/turtlebot_description/urdf/stacks/hexagons.urdf.xacro (robot description, xacro)
@@ -193,6 +193,7 @@
     <stack_top_pole parent="${parent}" number="2" x_loc="-0.0381" y_loc= "0.1505" z_loc="0.2920"/>
     <stack_top_pole parent="${parent}" number="3" x_loc="-0.0381" y_loc="-0.1505" z_loc="0.2920"/>
-    <stack_3d_sensor_pole parent="${parent}" number="0" x_loc="-0.1024" y_loc= "0.098" z_loc="0.2372"/>
-    <stack_3d_sensor_pole parent="${parent}" number="1" x_loc="-0.1024" y_loc="-0.098" z_loc="0.2372"/>
+    <!--stack_3d_sensor_pole parent="${parent}" number="0" x_loc="-0.1024" y_loc= "0.098" z_loc="0.2372"/-->
+ <stack_3d_sensor_pole parent="${parent}" number="0" x_loc="0" y_loc= "0.098" z_loc="0.2372"/>
+    <stack_3d_sensor_pole parent="${parent}" number="1" x_loc="0" y_loc="-0.098" z_loc="0.2372"/>
     <joint name="plate_top_joint" type="fixed">
       <origin xyz="-0.01364 0.0  0.3966" rpy="0 0 0"/>

File: turtlebot/turtlebot_description/urdf/turtlebot_properties.urdf.xacro (robot description, xacro)
@@ -19,5 +19,6 @@
      (currently in development and awaiting feedback)
    -->
-	<xacro:property name="cam_px" value="-0.087" />
+	<!--xacro:property name="cam_px" value="-0.087" /-->
+	<xacro:property name="cam_px" value="0.0154" />
 <!--	<xacro:property name="cam_py" value="-0.0125" /> Y varies for different configurations. get sets in sensors_urdf -->
 	<xacro:property name="cam_pz" value="0.2870" />
